File: rx/kicad/rx.sch (KiCad schematic (older format))
At the start: 4 parts, among them J1 TB003-500-P08BE, SW1 1825910-6

Commit message: preparing plots
Connections:
- net Power Supply/AC_NEUTRAL: no longer J1.4
- new net Switching/COM: J1.4
Changed lines of the file:
@@
 F4 "OUT_3" O L 3850 3100 50
 F5 "OUT_4" O L 3850 3200 50
-F6 "COM" O L 3850 3700 50
+F6 "COM" O L 3850 3300 50
 F7 "IN_1" I R 4750 2900 50
 F8 "IN_2" I R 4750 3000 50
 F9 "IN_3" I R 4750 3100 50
 F10 "IN_4" I R 4750 3200 50
+F11 "AC_LINE" I L 3850 3600 50
+F12 "AC_NEUTRAL" I L 3850 3700 50
 $EndSheet
 $Sheet
@@
 	3250 3600 3400 3600
 Wire Wire Line
-	3400 3600 3400 4300
+	3400 3600 3400 3700
 Wire Wire Line
 	3400 4300 3850 4300
@@
 	3850 4200 3550 4200
 Wire Wire Line
-	3550 4200 3550 3700
-Wire Wire Line
 	3550 3500 3250 3500
-Wire Wire Line
-	3850 3700 3550 3700
-Connection ~ 3550 3700
-Wire Wire Line
-	3550 3700 3550 3500
-Wire Wire Line
-	3400 3600 3400 3300
-Wire Wire Line
-	3400 3300 3250 3300
-Connection ~ 3400 3600
 NoConn ~ 3250 3400
 $Comp
@@
 F5 "Vss" O R 4750 4300 50
 $EndSheet
+Wire Wire Line
+	3550 3500 3550 3600
+Wire Wire Line
+	3850 3300 3250 3300
+Wire Wire Line
+	3850 3600 3550 3600
+Connection ~ 3550 3600
+Wire Wire Line
+	3550 3600 3550 4200
+Wire Wire Line
+	3850 3700 3400 3700
+Connection ~ 3400 3700
+Wire Wire Line
+	3400 3700 3400 4300
 $EndSCHEMATC
