File: rx/kicad/Logic.sch (KiCad schematic (older format))
At the start: 2 parts, among them J3 CONN_08LOCK, U5 PIC16F627A-I_P

Commit message: wip
Connections:
- net Data: now also U5.7 (RB1/RX/DT); no longer U5.8 (RB2/TX/CK)
Changed lines of the file:
@@
 $Descr A4 11693 8268
 encoding utf-8
-Sheet 4 5
+Sheet 3 5
 Title ""
 Date ""
@@
 Text HLabel 9150 4250 2    50   Output ~ 0
 ZONE_4
-Text HLabel 2950 4450 0    50   Input ~ 0
+Text HLabel 2950 4350 0    50   Input ~ 0
 Data
 Text HLabel 2950 4250 0    50   Input ~ 0
@@
 Wire Wire Line
 	2950 4150 3200 4150
-Wire Wire Line
-	2950 4450 3200 4450
 $Comp
 L rx:CONN_08LOCK J3
@@
 	2900 4050 3200 4050
 NoConn ~ 3200 3750
-NoConn ~ 3200 4350
 Wire Wire Line
 	3200 4250 2950 4250
 Wire Wire Line
 	3200 4550 2950 4550
+Wire Wire Line
+	3200 4350 2950 4350
+NoConn ~ 3200 4450
 $EndSCHEMATC
