File: rx/kicad/Switching.sch (KiCad schematic (older format))
At the start: 5 parts, among them K1 EC2-5NU, K2 EC2-5NU, K3 EC2-5NU, K4 EC2-5NU, U1 ULN2003AN

Commit message: preparing plots
Connections:
- net COM: now also K1.4 (5), K2.4 (5), K3.4 (5), K4.4 (5); no longer K1.6 (9), K2.6 (9), K3.6 (9), K4.6 (9)
- net AC_NEUTRAL: now reaches K1.3 (4)
- net AC_NEUTRAL: now also K2.3 (4), K3.3 (4), K4.3 (4)
- new net AC_LINE: K1.6 (9), K2.6 (9), K3.6 (9), K4.6 (9)
- no-connect marks 22 -> 14
Changed lines of the file:
@@
 $Descr A4 11693 8268
 encoding utf-8
-Sheet 3 5
+Sheet 2 5
 Title ""
 Date ""
@@
 Wire Wire Line
 	3750 4800 3600 4800
-$Comp
-L rx:EC2-5NU K4
-U 1 1 6012DEAD
-P 5400 5500
-F 0 "K4" H 4600 5887 60  0000 C CNN
-F 1 "EC2-5NU" H 4600 5781 60  0000 C CNN
-F 2 "rx:EC2-5NU" H 4600 5740 60  0001 C CNN
-F 3 "" H 5400 5500 60  0000 C CNN
-	1    5400 5500
-	1    0    0    -1
-$EndComp
 Wire Wire Line
 	3800 5800 3650 5800
 Wire Wire Line
 	3750 2700 3150 2700
-Wire Wire Line
-	3150 6200 2850 6200
 Wire Wire Line
 	3800 5700 3150 5700
 Connection ~ 3150 5700
 Wire Wire Line
-	3150 5700 3150 6200
+	3150 5700 3150 6050
 Wire Wire Line
 	3750 4700 3150 4700
@@
 Text HLabel 3650 5800 0    50   Output ~ 0
 OUT_4
-Text HLabel 2850 6200 0    50   Output ~ 0
+Text HLabel 5800 6050 2    50   Output ~ 0
 COM
 Text GLabel 2800 2500 0    50   Input ~ 0
@@
 NoConn ~ 3750 2600
 NoConn ~ 5350 2600
-NoConn ~ 5350 2700
-NoConn ~ 5350 2800
 NoConn ~ 3750 3600
 NoConn ~ 5350 3600
-NoConn ~ 5350 3700
-NoConn ~ 5350 3800
 NoConn ~ 5350 4600
-NoConn ~ 5350 4700
-NoConn ~ 5350 4800
 NoConn ~ 3750 4600
 NoConn ~ 3800 5600
 NoConn ~ 5400 5600
-NoConn ~ 5400 5700
-NoConn ~ 5400 5800
 Text GLabel 9200 3650 2    50   Input ~ 0
 Vss
@@
 NoConn ~ 8850 3850
 NoConn ~ 8850 3950
+Text HLabel 2850 6050 0    50   Input ~ 0
+AC_LINE
+$Comp
+L rx:EC2-5NU K4
+U 1 1 6012DEAD
+P 5400 5500
+F 0 "K4" H 4600 5887 60  0000 C CNN
+F 1 "EC2-5NU" H 4600 5781 60  0000 C CNN
+F 2 "rx:EC2-5NU" H 4600 5740 60  0001 C CNN
+F 3 "" H 5400 5500 60  0000 C CNN
+	1    5400 5500
+	1    0    0    -1
+$EndComp
+Wire Wire Line
+	5350 2800 5600 2800
+Wire Wire Line
+	5600 2800 5600 3800
+Wire Wire Line
+	5600 6050 5800 6050
+Wire Wire Line
+	5400 5800 5600 5800
+Connection ~ 5600 5800
+Wire Wire Line
+	5600 5800 5600 6050
+Wire Wire Line
+	5350 4800 5600 4800
+Connection ~ 5600 4800
+Wire Wire Line
+	5600 4800 5600 5800
+Wire Wire Line
+	5350 3800 5600 3800
+Connection ~ 5600 3800
+Wire Wire Line
+	5600 3800 5600 4800
+Wire Wire Line
+	2850 6050 3150 6050
+Text HLabel 5800 6200 2    50   Input ~ 0
+AC_NEUTRAL
+Wire Wire Line
+	5800 6200 5450 6200
+Wire Wire Line
+	5450 6200 5450 5700
+Wire Wire Line
+	5450 2700 5350 2700
+Wire Wire Line
+	5350 3700 5450 3700
+Connection ~ 5450 3700
+Wire Wire Line
+	5450 3700 5450 2700
+Wire Wire Line
+	5350 4700 5450 4700
+Connection ~ 5450 4700
+Wire Wire Line
+	5450 4700 5450 3700
+Wire Wire Line
+	5400 5700 5450 5700
+Connection ~ 5450 5700
+Wire Wire Line
+	5450 5700 5450 4700
 $EndSCHEMATC

Commit message: wip
Connections:
- net Vdd: now also K1.1, K2.1, K3.1, K4.1; no longer K1.8 (12), K2.8 (12), K3.8 (12), K4.8 (12)
- net at U1.13 (4C): now also K4.8 (12); no longer K1.1
- net at U1.14 (3C): now also K3.8 (12); no longer K2.1
- net at U1.15 (2C): now also K2.8 (12); no longer K3.1
- net at U1.16 (1C): now also K1.8 (12); no longer K4.1
Other:
- moved on the sheet: K1, K2, K3, K4, U1
