File: rx/kicad/rx.kicad_pcb (KiCad board)
At the start: 2 copper layers, 51 x 100 mm, 20 parts, among them J1 TB003-500-P08BE, J2 173010542, J3 CONN_08LOCK, J4 RF2-03E-T-00-50-G, K1 EC2-5NU, K2 EC2-5NU, K3 EC2-5NU, K4 EC2-5NU, M1 RF-LINK_RX, SW1 1825910-6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

Commit message: preparing plots
Parts:
- moved REF** 1.50 mm to (160.0, 101.0)
- moved U1 0.44 mm to (119.7, 110.6)
Connections:
- J1 pad 4: /Power Supply/AC_NEUTRAL -> /Switching/COM
- K1 pad 3: Net-(K1-Pad3) -> /Power Supply/AC_NEUTRAL
- K1 pad 4: Net-(K1-Pad4) -> /Switching/COM
- K2 pad 3: Net-(K2-Pad3) -> /Power Supply/AC_NEUTRAL
- K2 pad 4: Net-(K2-Pad4) -> /Switching/COM
- K3 pad 3: Net-(K3-Pad3) -> /Power Supply/AC_NEUTRAL
- K3 pad 4: Net-(K3-Pad4) -> /Switching/COM
- K4 pad 3: Net-(K4-Pad3) -> /Power Supply/AC_NEUTRAL
- K4 pad 4: Net-(K4-Pad4) -> /Switching/COM
Routing:
- net /Switching/COM: track 0.00 -> 99.8 mm
- net /Power Supply/AC_NEUTRAL: track 37.0 -> 91.8 mm
- net /Power Supply/AC_LINE: track 82.2 -> 83.8 mm
- net Net-(K1-Pad1): track 16.6 -> 17.5 mm
- net Net-(K4-Pad1): track 11.2 -> 11.9 mm
- net Net-(K2-Pad1): track 10.9 -> 11.4 mm
Other:
- rule pad_to_mask_clearance: 0.0508 -> 0

Commit message: wip
Connections:
- K1 pad 1: Net-(K1-Pad1) -> Vdd
- K1 pad 8: Vdd -> Net-(K1-Pad8)
- K2 pad 1: Net-(K2-Pad1) -> Vdd
- K2 pad 8: Vdd -> Net-(K2-Pad8)
- K3 pad 1: Net-(K3-Pad1) -> Vdd
- K3 pad 8: Vdd -> Net-(K3-Pad8)
- K4 pad 1: Net-(K4-Pad1) -> Vdd
- K4 pad 8: Vdd -> Net-(K4-Pad8)
- U1 pad 13: Net-(K1-Pad1) -> Net-(K4-Pad8)
- U1 pad 14: Net-(K2-Pad1) -> Net-(K3-Pad8)
- U1 pad 15: Net-(K3-Pad1) -> Net-(K2-Pad8)
- U1 pad 16: Net-(K4-Pad1) -> Net-(K1-Pad8)
- U5 pad 7: Net-(U5-Pad7) -> /Logic/Data
- U5 pad 8: /Logic/Data -> Net-(U5-Pad8)
Routing:
- net Net-(K4-Pad8): track 0.00 -> 34.1 mm
- net Net-(K3-Pad8): track 0.00 -> 23.3 mm
- net Net-(K1-Pad8): track 0.00 -> 21.9 mm
- net Net-(K2-Pad8): track 0.00 -> 21.7 mm
- net Net-(K1-Pad1): track 17.5 -> 0.00 mm
- net Net-(K4-Pad1): track 11.9 -> 0.00 mm
- net Net-(K2-Pad1): track 11.4 -> 0.00 mm
- net Net-(K3-Pad1): track 8.79 -> 0.00 mm
- net Net-(D2-Pad1): track 5.34 -> 8.91 mm
- net /Logic/Button: track 53.4 -> 50.5 mm
- net /Logic/Data: track 25.8 -> 28.3 mm
- net Vdd: track 164.5 -> 162.4 mm
- net /Switching/IN_3: track 42.3 -> 44.2 mm
- net /Power Supply/AC_NEUTRAL: track 91.8 -> 91.1 mm
