File: tx/kicad/Logic.sch (KiCad schematic (older format))
At the start: 2 parts, among them J3 CONN_08LOCK, U5 PIC16F627A-I_P

Commit message: wip
Connections:
- net Data: now also U5.8 (RB2/TX/CK); no longer U5.7 (RB1/RX/DT)
Changed lines of the file:
@@
 Text HLabel 9150 4250 2    50   Input ~ 0
 ZONE_4
-Text HLabel 2950 4350 0    50   Output ~ 0
+Text HLabel 2950 4450 0    50   Output ~ 0
 Data
 Text HLabel 2950 4250 0    50   Input ~ 0
@@
 Wire Wire Line
 	2950 4250 3200 4250
-Wire Wire Line
-	2950 4350 3200 4350
 Wire Wire Line
 	2950 4550 3200 4550
@@
 NoConn ~ 3200 3850
 NoConn ~ 3200 3950
-NoConn ~ 3200 4450
 NoConn ~ 5450 2000
 NoConn ~ 5550 2000
@@
 	2900 4050 3200 4050
 NoConn ~ 3200 3750
+Wire Wire Line
+	3200 4450 2950 4450
+NoConn ~ 3200 4350
 $EndSCHEMATC
