File: tx/kicad/tx.kicad_pcb (KiCad board)
At the start: 2 copper layers, 51 x 100 mm, 27 parts, among them J1 TB003-500-P08BE, J2 173010542, J3 CONN_08LOCK, J4 RF2-03E-T-00-50-G, M1 RF-LINK_TX, SW1 1825910-6, U1 H11L1M, U2 H11L1M, U3 H11L1M, U4 H11L1M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

Commit message: preparing plots
Parts:
- added REF**: OSHW-Logo2_7.3x6mm_SilkScreen, Symbol:OSHW-Logo2_7.3x6mm_SilkScreen, F.Cu at (144.5, 117.0)
- moved R1 3.61 mm to (146.0, 92.5)
Routing:
- net Net-(D1-Pad1): track 31.8 -> 32.6 mm
Other:
- rule pad_to_mask_clearance: 0.0508 -> 0
- board text added: "Copyright (C) Scuddles 2021"
- board text added: "Irrigation Wireless Relay"

Commit message: wip
Parts:
- moved REF** 2.50 mm to (146.0, 115.0)
Connections:
- net /Signal Conditioner/COMM renamed /Signal Conditioner/COM
- U5 pad 7: /Logic/Data -> Net-(U5-Pad7)
- U5 pad 8: Net-(U5-Pad8) -> /Logic/Data
Routing:
- net Vdd: track 182.8 -> 178.7 mm
- net Net-(D3-Pad1): track 4.30 -> 8.16 mm
- net /Logic/Data: track 26.9 -> 24.7 mm
Other:
- board text added: "Rev 1.2"
- board text added: "^"
