File: tx/kicad/tx.sch (KiCad schematic (older format))
At the start: 4 parts, among them J1 TB003-500-P08BE, SW1 1825910-6

Commit message: wip
Connections:
- net Signal Conditioner/COMM renamed Signal Conditioner/COM
Changed lines of the file:
@@
 F8 "OUT_3" O R 4800 3200 50
 F9 "OUT_4" O R 4800 3450 50
-F10 "COMM" O L 3950 3850 50
+F10 "COM" O L 3950 4100 50
 $EndSheet
 $Sheet
@@
 Wire Wire Line
 	3650 3450 3950 3450
-Wire Wire Line
-	2750 4100 3850 4100
-Wire Wire Line
-	3850 4100 3850 3850
-Wire Wire Line
-	3850 3850 3950 3850
 Text GLabel 4950 4750 2    50   UnSpc ~ 0
 Vdd
@@
 	-1   0    0    1
 $EndComp
+Wire Wire Line
+	2750 4100 3950 4100
 $EndSCHEMATC
